File: KiCAD Files/Buzzer PCB V2/Buzzer PCB.kicad_pcb (KiCad board)
At the start: 2 copper layers, 136.3 x 75.3 mm, 31 parts, among them J1 2600mAh LiPo JST-PH bottom, J10 SparkFun Thing Plus ESP32 WRO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, J11 M16968 OLED + Rotary Knob, J5 HGLRC M100 Mini GPS, J6 BMP581/BMP5xx top pads, J7 SHT41 top pads, Q1 S8050, Q2 S8050, Q3 S8050, SW1 SS12D00G5 power switch, U1 TP4057 USB-C charger, U2 Comidox 5V Booster

Commit message: Latest board
Routing:
- net /OLED_CONFIRM: track 60.9 -> 64.5 mm
Changed lines of the file:
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@@
 			(layer "F.SilkS")
 		)
-		(fp_text user "SPARKFUN THING PLUS ESP32 WROOM-C"
-			(at -28.845 -10.23 0)
+		(fp_text user "header geometry from SparkFun Eagle J5"
+			(at -28.845 0 0)
 			(layer "F.SilkS")
 			(effects
 				(font
-					(size 0.72 0.72)
+					(size 0.48 0.48)
 					(thickness 0.12)
 				)
 			)
 		)
-		(fp_text user "header geometry from SparkFun Eagle J5"
-			(at -28.845 0 0)
+		(fp_text user "USB-C end"
+			(at -28.845 10.23 0)
 			(layer "F.SilkS")
 			(effects
 				(font
-					(size 0.48 0.48)
+					(size 0.58 0.58)
 					(thickness 0.12)
 				)
 			)
 		)
-		(fp_text user "USB-C end"
-			(at -28.845 10.23 0)
+		(fp_text user "SPARKFUN THING PLUS ESP32 WROOM-C"
+			(at -25.75 -14 0)
 			(layer "F.SilkS")
 			(effects
 				(font
-					(size 0.58 0.58)
+					(size 0.72 0.72)
 					(thickness 0.12)
 				)
@@
 	)
 	(gr_text "J10 SparkFun Thing Plus ESP32 WROOM-C, SparkFun Eagle header geometry"
-		(at 67 58.95 0)
+		(at 74 55.75 0)
 		(layer "F.SilkS")
 		(effects
@@
 	)
 	(segment
+		(start 133.225 81.975)
+		(end 133.25 82)
+		(width 0.5)
+		(layer "F.Cu")
+		(net "/OLED_CONFIRM")
+	)
+	(segment
 		(start 99.75 81.5)
 		(end 99.75 76.25)
@@
 		(width 0.5)
 		(layer "F.Cu")
+		(net "/OLED_CONFIRM")
+	)
+	(segment
+		(start 133.225 78.41)
+		(end 133.225 81.975)
+		(width 0.5)
+		(layer "F.Cu")
