File: KiCAD Files/Buzzer PCB V2/Buzzer PCB.kicad_pcb (KiCad board)
At the start: 2 copper layers, 136.3 x 75.3 mm, 31 parts, among them J1 2600mAh LiPo JST-PH bottom, J10 SparkFun Thing Plus ESP32 WRO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, J11 M16968 OLED + Rotary Knob, J5 HGLRC M100 Mini GPS, J6 BMP581/BMP5xx top pads, J7 SHT41 top pads, Q1 S8050, Q2 S8050, Q3 S8050, SW1 SS12D00G5 power switch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

Commit message: getting close
Parts:
- moved C2 5.96 mm to (74.5, 90.0)
Routing:
- net /3V3: track 185.7 -> 195.1 mm
- net /GND: track 422.2 -> 428.6 mm
Other:
- board text removed: "BTN nets copied from Ant Display: BACK GPIO3, NEXT GPIO4, DOWN GPIO5, UP net on FREEBIE/ESP4"
- board text removed: "C1 bulk, C2 decoupling on SW_BAT/GND"
- board text removed: "J11 SparkFun Qwiic OLED 1.3in; J3 pins GND 3V3 SDA SCL"
- board text removed: "U1 USB-C edge faces board left; BAT pads face right"

Commit message: ready to mill
Parts:
- added H1: MountingHole_3.2mm_M3, MountingHole:MountingHole_3.2mm_M3, F.Cu at (61.5, 52.5)
- added H2: MountingHole_3.2mm_M3, MountingHole:MountingHole_3.2mm_M3, F.Cu at (61.5, 118.3)
- added H3: MountingHole_3.2mm_M3, MountingHole:MountingHole_3.2mm_M3, F.Cu at (193.0, 52.5)
- added H4: MountingHole_3.2mm_M3, MountingHole:MountingHole_3.2mm_M3, F.Cu at (193.0, 118.3)
- moved REF** 8.01 mm to (145.5, 54.6)
- moved ? 8.00 mm to (153.5, 54.6)
- moved U1 3.46 mm to (71.5, 111.2)
- moved R3 0.66 mm to (128.2, 52.9)
- moved ? 0.23 mm to (149.4, 54.6)
Connections:
- J10 pad 1: /SDA -> /GPS_TX_THING_RX
- J10 pad 14: /GPS_RX_THING_TX -> unconnected-(J10-TX_ESP17-Pad14)
- J10 pad 15: /GPS_TX_THING_RX -> unconnected-(J10-RX_ESP16-Pad15)
- J10 pad 2: /SCL -> /GPS_RX_THING_TX
- J10 pad 4: unconnected-(J10-GPIO5/ESP32-Pad4) -> /SCL
- J10 pad 6: unconnected-(J10-GPIO3/ESP33-Pad6) -> /SDA
- J5 pad 1: /GPS_RX_THING_TX -> /OLD_GPS_RX_UNUSED
- J5 pad 2: /GPS_TX_THING_RX -> /OLD_GPS_TX_UNUSED
- U2 pad 1: /BOOST_5V -> /SW_BAT
- U2 pad 3: /SW_BAT -> /BOOST_5V
Routing:
- net /BOOST_5V: track 90.5 -> 164.7 mm
- net /3V3: track 195.1 -> 161.3 mm
- net /GPS_TX_THING_RX: track 24.7 -> 0.00 mm
- net /BUZZER_BASE: track 169.4 -> 191.6 mm
- net /GPS_RX_THING_TX: track 20.4 -> 0.00 mm
- net /SW_BAT: track 115.4 -> 129.8 mm
- net /SDA: track 181.0 -> 169.6 mm
- net /GND: track 428.6 -> 439.5 mm
- net /SCL: track 169.1 -> 164.8 mm
- net /BAT_IN: track 22.7 -> 26.3 mm
- net /BUZZER_BASE2: track 181.8 -> 179.7 mm
- net /BUZZER_BASE3: track 141.4 -> 139.8 mm
- net /BTN_DOWN_GPIO5: track 47.8 -> 48.4 mm
- net /BUZZER3_GPIO2_ESP27: track 5.92 -> 5.32 mm
Other:
- board size 136.3 x 75.3 mm -> 140.7 x 74.9 mm

Commit message: DEEP CORNER HOLES
Parts:
- added ?: , , F.Cu at (174.5, 68.4)
- added ?: , , F.Cu at (173.0, 111.9)
- added ?: , , F.Cu at (159.8, 109.6)
- moved R1 1.15 mm to (123.0, 64.4)
Routing:
- net /3V3: track 161.3 -> 199.6 mm
- net /BUZZER_BASE2: track 179.7 -> 186.6 mm
- net /GND: track 439.5 -> 443.1 mm
- net /BUZZER_BASE: track 191.6 -> 188.4 mm
- net /BTN_BACK_GPIO3: track 17.0 -> 19.5 mm
- net /SW_BAT: track 129.8 -> 127.5 mm, vias 1 -> 0
- net /BTN_DOWN_GPIO5: track 48.4 -> 50.6 mm
- net /SCL: track 164.8 -> 163.2 mm
- net /BTN_UP_GPIO21: track 17.0 -> 18.6 mm
- net /BTN_NEXT_GPIO4: track 17.0 -> 18.5 mm
- net /D13_BUZZER_GPIO13: track 5.19 -> 6.34 mm
- net /SDA: track 169.6 -> 168.5 mm
- net /BUZZER2_ESP26: track 9.58 -> 10.4 mm
- net /BUZZER_BASE3: track 139.8 -> 140.5 mm
- net /BOOST_5V: vias 1 -> 0
