File: KiCAD Files/Buzzer PCB V2/Buzzer PCB.kicad_pcb (KiCad board)
At the start: 2 copper layers, 140.7 x 74.9 mm, 38 parts, among them J1 2600mAh LiPo JST-PH bottom, J10 SparkFun Thing Plus ESP32 WRO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, J11 M16968 OLED + Rotary Knob, J5 HGLRC M100 Mini GPS, J6 BMP581/BMP5xx top pads, J7 SHT41 top pads, Q1 S8050, Q2 S8050, Q3 S8050, SW1 SS12D00G5 power switch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

Commit message: REATTEMPT
Parts:
- removed the ? at (173.0, 111.9)
- removed the ? at (159.8, 109.6)
- added ?: , , F.Cu at (93.8, 81.8)
- SW1: value SS12D00G5 power switch -> SS12F44G3 power switch; footprint Button_Switch_THT:SS12D00G5_Custom -> Vario_Buzzer_V2:SS12F44G3_5.9x12.25_P3.00
- moved C1 5.77 mm to (76.1, 76.3)
- moved J1 5.20 mm to (63.4, 82.7)
- turned SW1 to 180 degrees
Connections:
- J1 pad 1: /BAT_IN -> /GND
- J1 pad 2: /GND -> /BAT_IN
- U1 pad 1: /BAT_IN -> /GND
- U1 pad 2: /GND -> /BAT_IN
Routing:
- net /3V3: track 199.6 -> 142.1 mm
- net /BOOST_5V: track 164.7 -> 192.8 mm
- net /SCL: track 163.2 -> 185.8 mm
- net /GND: track 443.1 -> 462.0 mm
- net /BAT_IN: track 26.3 -> 41.7 mm
- net /SDA: track 168.5 -> 179.4 mm
