File: KiCAD Files/Buzzer PCB V2/Buzzer PCB.kicad_sch (KiCad schematic)
At the start: 27 parts, among them J1 2600mAh LiPo JST-PH bottom, J10 SparkFun Thing Plus ESP32 WRO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, J11 M16968 OLED + Rotary Knob, J3 Optional SD module 18x18 swap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, J5 HGLRC M100 Mini GPS, J6 BMP581/BMP5xx top pads, J7 SHT41 top pads, Q1 S8050, Q2 S8050, Q3 S8050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

Commit message: pcb
Connections:
- net 3V3: now also C2.2, J10.27 (3V3), J3.6 (3V3), J5.3 (VCC); no longer J3.1 (GND), J5.2 (TX)
- net BAT_IN: now also J1.1 (+), U1.1 (BAT+); no longer J1.2 (-), U1.2 (BAT-)
- net BUZZER_LOW: now also BZ1.2 (-), D1.2 (A), Q1.3 (C); no longer BZ1.1 (+), BZ2.1 (+), BZ3.1 (+), D1.1 (K), D2.1 (K), D3.1 (K), Q1.1 (E), Q2.1 (E), Q3.1 (E)
- net D13_BUZZER_GPIO13: now also J10.9 (D13/ESP13_STAT); no longer J10.15 (RX_ESP16)
- net GND: now also J1.2 (-), J3.1 (GND), J5.4 (GND), Q1.1 (E), Q2.1 (E), Q3.1 (E), U1.2 (BAT-); no longer J1.1 (+), J3.6 (3V3), J5.1 (RX), Q1.3 (C), Q2.3 (C), Q3.3 (C), SW1.1 (ON), U1.1 (BAT+)
- net GPS_RX_THING_TX: now also J5.1 (RX); no longer J5.4 (GND)
- net GPS_TX_THING_RX: now also J10.15 (RX_ESP16), J5.2 (TX); no longer J10.9 (D13/ESP13_STAT), J5.3 (VCC)
- net SD_CS_GPIO2: now also J3.5 (CS); no longer J3.2 (MISO)
- net SPI_MISO: now also J3.2 (MISO); no longer J3.5 (CS)
- net SPI_MOSI: now also J3.4 (MOSI); no longer J3.3 (CLK)
- net SPI_SCK: now also J3.3 (CLK); no longer J3.4 (MOSI)
- removed net A: BZ1.2 (-), BZ2.2 (-), BZ3.2 (-), D1.2 (A), D2.2 (A), D3.2 (A), U2.3 (Vout)
- new net BOOST_5V: BZ1.1 (+), BZ2.1 (+), BZ3.1 (+), D1.1 (K), D2.1 (K), D3.1 (K), U2.3 (Vout)
- new net BUZZER_LOW2: BZ2.2 (-), D2.2 (A), Q2.3 (C)
- new net BUZZER_LOW3: BZ3.2 (-), D3.2 (A), Q3.3 (C)
- no-connect marks 6 -> 18

Commit message: updated pcb
Parts:
- removed J3: Optional SD module 18x18 swapped, Vario_Buzzer_V2:SD_Module_18x18_6Pin_Back, symbol Vario_Buzzer_V2:SD_Module_6_Swapped
Connections:
- net SD_CS_GPIO2: no longer names the net of J10.23 (A1/ESP25)
- net SPI_MISO: no longer names the net of J10.16 (MISO/POCI_ESP19)
- net SPI_MOSI: no longer names the net of J10.17 (MOSI/PICO_ESP23)
- net SPI_SCK: no longer names the net of J10.18 (SCK_ESP18)
- no-connect marks 18 -> 22
Other:
- note removed: "SparkFun Thing Plus pinout and module outline are from SparkFun Eagle hardware. Onboard microSD exists; J3 is optional external SPI SD using GPIO2 as CS."

Commit message: ready to mill
Connections:
- net GPS_RX_THING_TX: now also J10.2 (SCL/ESP22); no longer J10.14 (TX_ESP17), J5.1 (RX)
- net GPS_TX_THING_RX: now also J10.1 (SDA/ESP21); no longer J10.15 (RX_ESP16), J5.2 (TX)
- net SCL: now also J10.4 (GPIO5/ESP32); no longer J10.2 (SCL/ESP22)
- net SDA: now also J10.6 (GPIO3/ESP33); no longer J10.1 (SDA/ESP21)
- new net OLD_GPS_RX_UNUSED: J5.1 (RX)
- new net OLD_GPS_TX_UNUSED: J5.2 (TX)
Other:
- note added: "External M100 GPS plugs into SparkFun onboard Qwiic socket as UART: GPIO21/SDA=GPS TX into ESP RX, GPIO22/SCL=GPS RX from ESP TX."
- note added: "I2C bus moved off SparkFun Qwiic pins: SDA uses ESP33, SCL uses ESP32; onboard legacy M100 footprint nets are unused."
- note added: "SparkFun Thing Plus and M16968 OLED/rotary module replace the Feather/FeatherWing. OLED/SHT/BMP share relocated SDA/SCL; rotary controls replace standalone tactile switches."
- note removed: "HGLRC M100 footprint uses manual pad order RX TX VCC GND; VCC is tied to 3V3 per HGLRC 3.3V-5V product spec."
- note removed: "M16968 rotary button/encoder net names replace standalone tactile switches; PUSH/UP is routed to Thing FREEBIE/ESP4 to keep SDA free for I2C."
- note removed: "SparkFun Thing Plus and M16968 OLED/rotary module replace the Feather/FeatherWing. OLED uses direct 3V3/GND/SDA/SCL pads; rotary controls replace standalone tactile switches."
Changed lines of the file:
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@@
 		(comment 1 "SparkFun Thing Plus + M16968 OLED/rotary replacement; placement only, no traces")
 	)
-	(text "HGLRC M100 footprint uses manual pad order RX TX VCC GND; VCC is tied to 3V3 per HGLRC 3.3V-5V product spec."
+	(text "External M100 GPS plugs into SparkFun onboard Qwiic socket as UART: GPIO21/SDA=GPS TX into ESP RX, GPIO22/SCL=GPS RX from ESP TX."
 		(exclude_from_sim no)
 		(at 76.01 60.9 0)
@@
 		)
 	)
-	(text "M16968 rotary button/encoder net names replace standalone tactile switches; PUSH/UP is routed to Thing FREEBIE/ESP4 to keep SDA free for I2C."
+	(text "I2C bus moved off SparkFun Qwiic pins: SDA uses ESP33, SCL uses ESP32; onboard legacy M100 footprint nets are unused."
 		(exclude_from_sim no)
 		(at 76.01 54.9 0)
@@
 		)
 	)
-	(text "SparkFun Thing Plus and M16968 OLED/rotary module replace the Feather/FeatherWing. OLED uses direct 3V3/GND/SDA/SCL pads; rotary controls replace standalone tactile switches."
+	(text "SparkFun Thing Plus and M16968 OLED/rotary module replace the Feather/FeatherWing. OLED/SHT/BMP share relocated SDA/SCL; rotary controls replace standalone tactile switches."
 		(exclude_from_sim no)
 		(at 76.01 42.9 0)
@@
 	)
 	(no_connect
-		(at 93.98 133.35)
+		(at 36.83 146.05)
 	)
 	(no_connect
@@
 	)
 	(no_connect
+		(at 36.83 148.59)
+	)
+	(no_connect
 		(at 36.83 138.43)
 	)
@@
 	)
 	(no_connect
-		(at 93.98 138.43)
-	)
-	(no_connect
 		(at 225.31 119.25)
 	)
@@
 	(wire
 		(pts
-			(xy 24.13 146.05) (xy 36.83 146.05)
+			(xy 102.87 133.35) (xy 93.98 133.35)
 		)
 		(stroke
@@
 	(wire
 		(pts
-			(xy 24.13 148.59) (xy 36.83 148.59)
+			(xy 102.87 138.43) (xy 93.98 138.43)
 		)
 		(stroke
@@
 		)
 	)
-	(label "GPS_RX_THING_TX"
-		(at 24.13 148.59 0)
+	(label "SDA"
+		(at 102.87 133.35 0)
 		(effects
 			(font
@@
 		)
 	)
-	(label "SDA"
+	(label "GPS_TX_THING_RX"
 		(at 31.75 133.35 0)
 		(effects
@@
 		)
 	)
-	(label "GPS_TX_THING_RX"
-		(at 24.13 146.05 0)
+	(label "SCL"
+		(at 102.87 138.43 0)
 		(effects
 			(font
@@
 		)
 	)
-	(label "SCL"
+	(label "GPS_RX_THING_TX"
 		(at 31.75 135.89 0)
 		(effects
@@
 		)
 	)
-	(label "GPS_TX_THING_RX"
+	(label "OLD_GPS_TX_UNUSED"
 		(at 220.23 81.63 0)
 		(effects
@@
 		)
 	)
-	(label "GPS_RX_THING_TX"
+	(label "OLD_GPS_RX_UNUSED"
 		(at 220.23 79.09 0)
 		(effects

Commit message: REATTEMPT
Parts:
- SW1: value SS12D00G5 power switch -> SS12F44G3 power switch; footprint Button_Switch_THT:SS12D00G5_Custom -> Vario_Buzzer_V2:SS12F44G3_5.9x12.25_P3.00
Changed lines of the file:
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@@
 			)
 		)
-		(property "Value" "SS12D00G5 power switch"
+		(property "Value" "SS12F44G3 power switch"
 			(at 47.4 89.4 0)
 			(show_name no)
@@
 			)
 		)
-		(property "Footprint" "Button_Switch_THT:SS12D00G5_Custom"
+		(property "Footprint" "Vario_Buzzer_V2:SS12F44G3_5.9x12.25_P3.00"
 			(at 47.4 95.75 0)
 			(hide yes)
