File: KiCAD Files/Buzzer PCB V3 (rerouting traces)/Buzzer PCB V3 (rerouted traces)/Buzzer PCB V3 (rerouted traces).kicad_pcb (KiCad board)
At the start: 2 copper layers, 140.7 x 74.9 mm, 51 parts, among them J1 2600mAh LiPo JST-PH bottom, J10 SparkFun Thing Plus ESP32 WRO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, J11 M16968 OLED + Rotary Knob, J5 HGLRC M100 Mini GPS, J6 BMP581/BMP5xx top pads, J7 SHT41 top pads, Q1 S8050, Q2 S8050, Q3 S8050, SW1 SS12F44G3 power switch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

Commit message: FInal Sparkfun Version
Parts:
- removed the ? at (155.5, 105.0)
- removed the ? at (151.5, 113.8)
- removed the ? at (174.5, 68.4)
- added ?: , , F.Cu at (165.8, 105.0)
- added ?: , , F.Cu at (107.5, 65.2)
- added ?: , , F.Cu at (165.8, 119.2)
- C1, C2: moved to B.Cu
- J7: value SHT41 top pads -> SHT41 mechanical only
- R1, R1-1, R1-2, R1-3, R2, R3: moved to F.Cu
- moved ? 37.1 mm to (127.0, 90.5)
- moved BZ2 36.9 mm to (177.8, 112.2)
- moved J6 34.8 mm to (123.2, 103.4), turned to 0 degrees
- moved REF** 32.6 mm to (182.8, 62.7)
- moved R5 29.2 mm to (93.3, 66.5), turned to 0 degrees
- moved BZ3 26.1 mm to (177.8, 97.8)
- moved D2 24.8 mm to (185.3, 111.9)
- moved ? 24.1 mm to (132.0, 90.5)
- moved Q2 22.6 mm to (170.5, 119.3)
- moved ? 21.5 mm to (165.8, 90.5)
- moved Q3 18.7 mm to (170.5, 105.1)
- moved BZ1 14.3 mm to (177.8, 83.6)
- moved J7 13.9 mm to (153.0, 98.7), turned to -90 degrees
- moved R4 12.5 mm to (103.5, 63.2), turned to 180 degrees
- moved D1 12.5 mm to (185.3, 83.4)
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Connections:
- ? pad 1: /BOOST_5V -> /GND
- J1 pad 1: /GND -> /BAT_IN
- J1 pad 2: /BAT_IN -> /GND
- R4 pad 1: /SW_BAT -> /VBAT_SENSE_A1
- R4 pad 2: /VBAT_SENSE_A1 -> /SW_BAT
- R5 pad 1: /VBAT_SENSE_A1 -> /GND
- R5 pad 2: /GND -> /VBAT_SENSE_A1
- U1 pad 1: /GND -> /BAT_IN
- U1 pad 2: /BAT_IN -> /GND
Routing:
- net /BUZZER_BASE: track 188.4 -> 79.5 mm
- net /SCL: track 186.4 -> 99.5 mm
- net /BOOST_5V: track 217.7 -> 135.3 mm
- net /BUZZER_BASE2: track 186.3 -> 109.6 mm
- net /GND: track 511.9 -> 452.5 mm
- net /SDA: track 179.4 -> 127.4 mm
- net /BUZZER_BASE3: track 140.5 -> 94.6 mm
- net /3V3: track 162.3 -> 131.4 mm
- net /BAT_IN: track 73.3 -> 56.4 mm
- net /BUZZER_LOW: track 24.4 -> 12.8 mm
- net /VBAT_SENSE_A1: track 12.2 -> 23.4 mm
- net /BUZZER_LOW3: track 23.8 -> 12.7 mm
- net /BUZZER_LOW2: track 22.7 -> 12.6 mm
- net /SW_BAT: track 159.1 -> 163.3 mm
- net /OLED_CONFIRM: track 64.5 -> 68.1 mm
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