File: KiCAD Files/Buzzer PCB V3 (rerouting traces)/Buzzer PCB V3 (rerouted traces)/Buzzer PCB V3 (rerouted traces).kicad_pcb (KiCad board)
At the start: 2 copper layers, 140.7 x 74.9 mm, 51 parts, among them J1 2600mAh LiPo JST-PH bottom, J10 SparkFun Thing Plus ESP32 WRO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, J11 M16968 OLED + Rotary Knob, J5 HGLRC M100 Mini GPS, J6 BMP581/BMP5xx top pads, J7 SHT41 mechanical only, Q1 S8050, Q2 S8050, Q3 S8050, SW1 SS12F44G3 power switch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

Commit message: final
Parts:
- added ?: , , F.Cu at (133.2, 54.0)
- added ?: , , F.Cu at (69.0, 103.0)
- moved R4 1.58 mm to (104.0, 61.8)
- moved R3 1.35 mm to (128.2, 54.2)
- moved R5 1.01 mm to (93.5, 67.5)
- moved ? 0.56 mm to (99.8, 72.0)
- moved R1 0.08 mm to (123.1, 65.5)
Routing:
- net /SDA: track 127.4 -> 110.7 mm
- net /BAT_IN: track 56.4 -> 40.3 mm
- net /D13_BUZZER_GPIO13: track 14.9 -> 7.53 mm
- net /BUZZER3_GPIO2_ESP27: track 10.6 -> 4.22 mm
- net /BUZZER_BASE3: track 94.6 -> 98.8 mm
- net /GND: track 452.5 -> 454.7 mm
- net /SW_BAT: track 163.3 -> 161.2 mm
